File: 3v3-5v_regulator.kicad_pcb (KiCad board)
At the start: 2 copper layers, 39.1 x 20.2 mm, 8 parts, among them J1 USB_B_Micro, J2 Screw_Terminal_01x02, U1 AMS1117CD-3.3

Commit message: pcb done
Parts:
- moved C3 1.90 mm to (161.9, 137.3)
- moved C1 0.24 mm to (161.8, 132.1)
Routing:
- net GND: track 0.00 -> 1.53 mm, vias 0 -> 98
- added copper zone on F.Cu, net +3.3V
- added copper zone on F.Cu, net GND
Other:
- board size 39.1 x 20.2 mm -> 39.8 x 20.6 mm
- board text added: "5V-3.3V regulator"
