File: 3v3-5v_regulator.kicad_sch (KiCad schematic)
At the start: 8 parts, among them J1 USB_B_Micro, J2 Screw_Terminal_01x02, U1 AMS1117CD-3.3

Commit message: pcb done
Other:
- note added: "Dla 100nF 0402 - mniejsze, muszą być jak najbliżej U1 - sprzęgają wysokie Freq do masy Dla 22uF większe - magazyny energii, stabilizacja napięcia przy skokach poboru prądu."
- note added: "GND Fill Zone, żeby: - zmniejszyć rezystancję. - filtrować - 2 warstwy miedzi działają jak kondensator - oddawanie ciepła - łatwiejsza fabrykacja, bo nie trzeba usuwać miedzi kwasem"
- note added: "Thermal relief: - łatwe lutowanie - 4 mostki na pad - zapobiega odprowadzaniu ciepła z lutownicy - wyższa indukcyjność i rezystancja - standard THT Solid: - trudne lutowanie - do padów odprowadzających ciepło"
- note removed: "Dla 100nF 0402 - mniejsze, muszą być jak najbliżej U1. Dla 22uF większe."
Changed lines of the file:
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@@
 	(generator_version "10.0")
 	(paper "A4")
-	(text "Dla 100nF 0402 - mniejsze, muszą być jak najbliżej U1.\nDla 22uF większe."
+	(text "GND Fill Zone, żeby:\n- zmniejszyć rezystancję.\n- filtrować - 2 warstwy miedzi działają jak kondensator\n- oddawanie ciepła\n- łatwiejsza fabrykacja, bo nie trzeba usuwać miedzi kwasem"
+		(exclude_from_sim no)
+		(at 166.624 115.062 0)
+		(effects
+			(font
+				(size 1.27 1.27)
+			)
+		)
+	)
+	(text "Dla 100nF 0402 - mniejsze, muszą być jak najbliżej U1 - sprzęgają wysokie Freq do masy\nDla 22uF większe - magazyny energii, stabilizacja napięcia przy skokach poboru prądu.\n"
 		(exclude_from_sim no)
 		(at 153.67 87.63 0)
 		(effects
 			(font
+				(size 1.27 1.27)
+			)
+		)
+	)
+	(text "Thermal relief:\n- łatwe lutowanie\n- 4 mostki na pad - zapobiega odprowadzaniu ciepła z lutownicy\n- wyższa indukcyjność i rezystancja\n- standard THT\n\nSolid:\n- trudne lutowanie\n- do padów odprowadzających ciepło"
+		(exclude_from_sim no)
+		(at 165.608 132.842 0)
+		(effects
+			(font
